File: Electronics/KiCad/BackcoverMboard/Multiboard/Multiboard.sch (KiCad schematic (older format))
At the start: 7 parts, among them J1 Conn_01x05, J2 Conn_01x05_Male, J3 Conn_01x05_Male, J4 Conn_01x05, J5 USB_A, J6 USB_A, U1 FP-Back-Con

Commit message: added gcode and an updated board for ideal positioning of my Intenso HC 20000
Parts:
- J1, J4: footprint Fairphone-Back:Pad 01x05 -> Connector_PinHeader_2.54mm:PinHeader_1x05_P2.54mm_Vertical
- J2, J3: footprint Connector_PinHeader_2.54mm:PinHeader_1x05_P2.54mm_Vertical -> Fairphone-Back:Pad 01x05
- U1: symbol FP-Back:FP-Back-Con -> Multiboard-rescue:FP-Back-Con-FP-Back
Connections:
- net at U1.4 (D+): now also J1.3 (Pin_3); no longer J1.4 (Pin_4)
- net at U1.5 (D-): now also J1.4 (Pin_4); no longer J1.3 (Pin_3)
- net at J6.2 (D-): now also J4.4 (Pin_4), J5.2 (D-); no longer J4.3 (Pin_3)
- net at J6.3 (D+): now also J4.3 (Pin_3), J5.3 (D+); no longer J4.4 (Pin_4)
Changed lines of the file:
@@
 $EndDescr
 $Comp
-L FP-Back:FP-Back-Con U1
+L Multiboard-rescue:FP-Back-Con-FP-Back U1
 U 1 1 5D8F35EC
 P 1100 1200
@@
 F 0 "J1" H 1930 1092 50  0000 L CNN
 F 1 "Conn_01x05" H 1930 1001 50  0000 L CNN
-F 2 "Fairphone-Back:Pad 01x05" H 1850 1050 50  0001 C CNN
+F 2 "Connector_PinHeader_2.54mm:PinHeader_1x05_P2.54mm_Vertical" H 1850 1050 50  0001 C CNN
 F 3 "~" H 1850 1050 50  0001 C CNN
 	1    1850 1050
@@
 	1400 850  1650 850
 Wire Wire Line
-	1350 1050 1450 1050
-Wire Wire Line
-	1450 1050 1450 950
-Wire Wire Line
 	1450 950  1650 950
 Wire Wire Line
-	1350 1150 1500 1150
-Wire Wire Line
-	1500 1150 1500 1050
-Wire Wire Line
-	1500 1050 1650 1050
-Wire Wire Line
 	1350 1250 1550 1250
-Wire Wire Line
-	1550 1250 1550 1150
-Wire Wire Line
-	1550 1150 1650 1150
 $Comp
 L Connector:Conn_01x05_Male J2
@@
 F 0 "J2" H 2658 1431 50  0000 C CNN
 F 1 "Conn_01x05_Male" H 2658 1340 50  0000 C CNN
-F 2 "Connector_PinHeader_2.54mm:PinHeader_1x05_P2.54mm_Vertical" H 2550 1050 50  0001 C CNN
+F 2 "Fairphone-Back:Pad 01x05" H 2550 1050 50  0001 C CNN
 F 3 "~" H 2550 1050 50  0001 C CNN
 	1    2550 1050
-	1    0    0    -1
-$EndComp
-$Comp
-L Connector:USB_A J6
-U 1 1 5D8F76B3
-P 5100 900
-F 0 "J6" H 5157 1367 50  0000 C CNN
-F 1 "USB_A" H 5157 1276 50  0000 C CNN
-F 2 "Connector_USB:USB_A_Stewart_SS-52100-001_Horizontal" H 5250 850 50  0001 C CNN
-F 3 " ~" H 5250 850 50  0001 C CNN
-	1    5100 900
 	1    0    0    -1
 $EndComp
@@
 F 0 "J4" H 3768 575 50  0000 C CNN
 F 1 "Conn_01x05" H 3768 666 50  0000 C CNN
-F 2 "Fairphone-Back:Pad 01x05" H 3850 1000 50  0001 C CNN
+F 2 "Connector_PinHeader_2.54mm:PinHeader_1x05_P2.54mm_Vertical" H 3850 1000 50  0001 C CNN
 F 3 "~" H 3850 1000 50  0001 C CNN
 	1    3850 1000
@@
 F 0 "J3" H 3108 1481 50  0000 C CNN
 F 1 "Conn_01x05_Male" H 3108 1390 50  0000 C CNN
-F 2 "Connector_PinHeader_2.54mm:PinHeader_1x05_P2.54mm_Vertical" H 3000 1100 50  0001 C CNN
+F 2 "Fairphone-Back:Pad 01x05" H 3000 1100 50  0001 C CNN
 F 3 "~" H 3000 1100 50  0001 C CNN
 	1    3000 1100
@@
 	4050 800  5400 800
 Wire Wire Line
-	5400 800  5400 700
-Wire Wire Line
-	4050 900  5400 900
-Wire Wire Line
-	4050 1000 5400 1000
+	4050 1000 4550 1000
 Wire Wire Line
 	4050 1100 4200 1100
@@
 Wire Wire Line
 	4200 1100 5100 1100
+Wire Wire Line
+	1450 1050 1450 950
+Wire Wire Line
+	1350 1050 1450 1050
+Wire Wire Line
+	1350 1150 1650 1150
+Wire Wire Line
+	1550 1250 1550 1050
+Wire Wire Line
+	1550 1050 1650 1050
+Wire Wire Line
+	5400 800  5400 700
+$Comp
+L Connector:USB_A J6
+U 1 1 5D8F76B3
+P 5100 900
+F 0 "J6" H 5157 1367 50  0000 C CNN
+F 1 "USB_A" H 5157 1276 50  0000 C CNN
+F 2 "Connector_USB:USB_A_Stewart_SS-52100-001_Horizontal" H 5250 850 50  0001 C CNN
+F 3 " ~" H 5250 850 50  0001 C CNN
+	1    5100 900
+	1    0    0    -1
+$EndComp
+Wire Wire Line
+	4650 900  4650 1050
+Wire Wire Line
+	4650 1050 5400 1050
+Wire Wire Line
+	5400 1050 5400 1000
+Wire Wire Line
+	4550 1000 4550 950
+Wire Wire Line
+	4550 950  5400 950
+Wire Wire Line
+	5400 950  5400 900
+Wire Wire Line
+	4650 1050 4650 2050
+Connection ~ 4650 1050
+Wire Wire Line
+	4350 2050 4650 2050
+Wire Wire Line
+	4050 900  4650 900
+Wire Wire Line
+	4550 1000 4550 1950
+Wire Wire Line
+	4350 1950 4550 1950
+Connection ~ 4550 1000
 $EndSCHEMATC
